File: Standardized Subsheets/LDO.kicad_sch (KiCad schematic)
At the start: 3 parts, among them U1 AMS1117-3.3

Commit message: gitignore
Parts:
- renumbered C1 to C21, C2 to C22, U1 to U7
Changed lines of the file:
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@@
   (symbol (lib_id "power:GND") (at 96.52 91.44 0) (unit 1)
     (in_bom yes) (on_board yes) (fields_autoplaced)
-    (property "Reference" "#PWR01" (id 0) (at 96.52 97.79 0)
+    (property "Reference" "#PWR063" (id 0) (at 96.52 97.79 0)
       (effects (font (size 1.27 1.27)) hide)
     )
@@
   (symbol (lib_id "Device:C") (at 123.19 87.63 0) (unit 1)
     (in_bom yes) (on_board yes) (fields_autoplaced)
-    (property "Reference" "C2" (id 0) (at 127 86.3599 0)
+    (property "Reference" "C22" (id 0) (at 127 86.3599 0)
       (effects (font (size 1.27 1.27)) (justify left))
     )
@@
   (symbol (lib_id "power:GND") (at 111.76 91.44 0) (unit 1)
     (in_bom yes) (on_board yes) (fields_autoplaced)
-    (property "Reference" "#PWR02" (id 0) (at 111.76 97.79 0)
+    (property "Reference" "#PWR064" (id 0) (at 111.76 97.79 0)
       (effects (font (size 1.27 1.27)) hide)
     )
@@
   (symbol (lib_id "power:GND") (at 123.19 91.44 0) (unit 1)
     (in_bom yes) (on_board yes) (fields_autoplaced)
-    (property "Reference" "#PWR03" (id 0) (at 123.19 97.79 0)
+    (property "Reference" "#PWR065" (id 0) (at 123.19 97.79 0)
       (effects (font (size 1.27 1.27)) hide)
     )
@@
   (symbol (lib_id "Device:C") (at 96.52 87.63 0) (unit 1)
     (in_bom yes) (on_board yes) (fields_autoplaced)
-    (property "Reference" "C1" (id 0) (at 100.33 86.3599 0)
+    (property "Reference" "C21" (id 0) (at 100.33 86.3599 0)
       (effects (font (size 1.27 1.27)) (justify left))
     )
@@
   (symbol (lib_id "Regulator_Linear:AMS1117-3.3") (at 111.76 83.82 0) (unit 1)
     (in_bom yes) (on_board yes) (fields_autoplaced)
-    (property "Reference" "U1" (id 0) (at 111.76 76.2 0))
+    (property "Reference" "U7" (id 0) (at 111.76 76.2 0))
     (property "Value" "AMS1117-3.3" (id 1) (at 111.76 78.74 0))
     (property "Footprint" "Package_TO_SOT_SMD:SOT-223-3_TabPin2" (id 2) (at 111.76 78.74 0)

Commit message: Probably will be breaking everything
Parts:
- renumbered C21 to C7, C22 to C8, U7 to U2
Changed lines of the file:
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@@
   (symbol (lib_id "power:GND") (at 96.52 91.44 0) (unit 1)
     (in_bom yes) (on_board yes) (fields_autoplaced)
-    (property "Reference" "#PWR063" (id 0) (at 96.52 97.79 0)
+    (property "Reference" "#PWR026" (id 0) (at 96.52 97.79 0)
       (effects (font (size 1.27 1.27)) hide)
     )
@@
   (symbol (lib_id "Device:C") (at 123.19 87.63 0) (unit 1)
     (in_bom yes) (on_board yes) (fields_autoplaced)
-    (property "Reference" "C22" (id 0) (at 127 86.3599 0)
+    (property "Reference" "C8" (id 0) (at 127 86.3599 0)
       (effects (font (size 1.27 1.27)) (justify left))
     )
@@
   (symbol (lib_id "power:GND") (at 111.76 91.44 0) (unit 1)
     (in_bom yes) (on_board yes) (fields_autoplaced)
-    (property "Reference" "#PWR064" (id 0) (at 111.76 97.79 0)
+    (property "Reference" "#PWR027" (id 0) (at 111.76 97.79 0)
       (effects (font (size 1.27 1.27)) hide)
     )
@@
   (symbol (lib_id "power:GND") (at 123.19 91.44 0) (unit 1)
     (in_bom yes) (on_board yes) (fields_autoplaced)
-    (property "Reference" "#PWR065" (id 0) (at 123.19 97.79 0)
+    (property "Reference" "#PWR028" (id 0) (at 123.19 97.79 0)
       (effects (font (size 1.27 1.27)) hide)
     )
@@
   (symbol (lib_id "Device:C") (at 96.52 87.63 0) (unit 1)
     (in_bom yes) (on_board yes) (fields_autoplaced)
-    (property "Reference" "C21" (id 0) (at 100.33 86.3599 0)
+    (property "Reference" "C7" (id 0) (at 100.33 86.3599 0)
       (effects (font (size 1.27 1.27)) (justify left))
     )
@@
   (symbol (lib_id "Regulator_Linear:AMS1117-3.3") (at 111.76 83.82 0) (unit 1)
     (in_bom yes) (on_board yes) (fields_autoplaced)
-    (property "Reference" "U7" (id 0) (at 111.76 76.2 0))
+    (property "Reference" "U2" (id 0) (at 111.76 76.2 0))
     (property "Value" "AMS1117-3.3" (id 1) (at 111.76 78.74 0))
     (property "Footprint" "Package_TO_SOT_SMD:SOT-223-3_TabPin2" (id 2) (at 111.76 78.74 0)
