File: Standardized Subsheets/vrmsv2.kicad_sch (KiCad schematic)
At the start: 5 parts

Commit message: gitignore
Parts:
- renumbered D1 to D4, D2 to D5, D3 to D6, R1 to R21
Changed lines of the file:
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@@
   (symbol (lib_id "Device:D_Schottky") (at 78.74 45.72 180) (unit 1)
     (in_bom yes) (on_board yes) (fields_autoplaced)
-    (property "Reference" "D2" (id 0) (at 79.0575 41.91 0))
+    (property "Reference" "D5" (id 0) (at 79.0575 41.91 0))
     (property "Value" "0.7dV" (id 1) (at 79.0575 41.91 0)
       (effects (font (size 1.27 1.27)) hide)
@@
   (symbol (lib_id "power:+3V3") (at 151.13 36.83 0) (unit 1)
     (in_bom yes) (on_board yes) (fields_autoplaced)
-    (property "Reference" "#PWR0101" (id 0) (at 151.13 40.64 0)
+    (property "Reference" "#PWR050" (id 0) (at 151.13 40.64 0)
       (effects (font (size 1.27 1.27)) hide)
     )
@@
   (symbol (lib_id "power:+5V") (at 115.57 36.83 0) (unit 1)
     (in_bom yes) (on_board yes) (fields_autoplaced)
-    (property "Reference" "#PWR0102" (id 0) (at 115.57 40.64 0)
+    (property "Reference" "#PWR049" (id 0) (at 115.57 40.64 0)
       (effects (font (size 1.27 1.27)) hide)
     )
@@
   (symbol (lib_id "power:GND") (at 68.58 54.61 0) (unit 1)
     (in_bom yes) (on_board yes) (fields_autoplaced)
-    (property "Reference" "#PWR0103" (id 0) (at 68.58 60.96 0)
+    (property "Reference" "#PWR047" (id 0) (at 68.58 60.96 0)
       (effects (font (size 1.27 1.27)) hide)
     )
@@
   (symbol (lib_id "power:+24V") (at 50.8 45.72 0) (unit 1)
     (in_bom yes) (on_board yes) (fields_autoplaced)
-    (property "Reference" "#PWR0107" (id 0) (at 50.8 49.53 0)
+    (property "Reference" "#PWR046" (id 0) (at 50.8 49.53 0)
       (effects (font (size 1.27 1.27)) hide)
     )
@@
   (symbol (lib_id "Device:D_Zener") (at 68.58 49.53 270) (unit 1)
     (in_bom yes) (on_board yes) (fields_autoplaced)
-    (property "Reference" "D1" (id 0) (at 71.12 48.2599 90)
+    (property "Reference" "D4" (id 0) (at 71.12 48.2599 90)
       (effects (font (size 1.27 1.27)) (justify left))
     )
@@
   (symbol (lib_id "Device:LED") (at 83.82 53.34 90) (unit 1)
     (in_bom yes) (on_board yes) (fields_autoplaced)
-    (property "Reference" "D3" (id 0) (at 87.63 53.6574 90)
+    (property "Reference" "D6" (id 0) (at 87.63 53.6574 90)
       (effects (font (size 1.27 1.27)) (justify right))
     )
@@
   (symbol (lib_id "Device:R") (at 83.82 60.96 180) (unit 1)
     (in_bom yes) (on_board yes)
-    (property "Reference" "R1" (id 0) (at 86.36 60.96 90))
+    (property "Reference" "R21" (id 0) (at 86.36 60.96 90))
     (property "Value" "470R" (id 1) (at 88.9 60.96 90))
     (property "Footprint" "Resistor_SMD:R_0603_1608Metric_Pad0.98x0.95mm_HandSolder" (id 2) (at 85.598 60.96 90)
@@
   (symbol (lib_id "power:GND") (at 83.82 64.77 0) (unit 1)
     (in_bom yes) (on_board yes) (fields_autoplaced)
-    (property "Reference" "#PWR0108" (id 0) (at 83.82 71.12 0)
+    (property "Reference" "#PWR048" (id 0) (at 83.82 71.12 0)
       (effects (font (size 1.27 1.27)) hide)
     )

Commit message: Probably will be breaking everything
Parts:
- renumbered D4 to D5, D5 to D6, D6 to D7, R21 to R5
Changed lines of the file:
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@@
   (symbol (lib_id "Device:D_Schottky") (at 78.74 45.72 180) (unit 1)
     (in_bom yes) (on_board yes) (fields_autoplaced)
-    (property "Reference" "D5" (id 0) (at 79.0575 41.91 0))
+    (property "Reference" "D6" (id 0) (at 79.0575 41.91 0))
     (property "Value" "0.7dV" (id 1) (at 79.0575 41.91 0)
       (effects (font (size 1.27 1.27)) hide)
@@
   (symbol (lib_id "power:+3V3") (at 151.13 36.83 0) (unit 1)
     (in_bom yes) (on_board yes) (fields_autoplaced)
-    (property "Reference" "#PWR050" (id 0) (at 151.13 40.64 0)
+    (property "Reference" "#PWR025" (id 0) (at 151.13 40.64 0)
       (effects (font (size 1.27 1.27)) hide)
     )
@@
   (symbol (lib_id "power:+5V") (at 115.57 36.83 0) (unit 1)
     (in_bom yes) (on_board yes) (fields_autoplaced)
-    (property "Reference" "#PWR049" (id 0) (at 115.57 40.64 0)
+    (property "Reference" "#PWR024" (id 0) (at 115.57 40.64 0)
       (effects (font (size 1.27 1.27)) hide)
     )
@@
   (symbol (lib_id "power:GND") (at 68.58 54.61 0) (unit 1)
     (in_bom yes) (on_board yes) (fields_autoplaced)
-    (property "Reference" "#PWR047" (id 0) (at 68.58 60.96 0)
+    (property "Reference" "#PWR022" (id 0) (at 68.58 60.96 0)
       (effects (font (size 1.27 1.27)) hide)
     )
@@
   (symbol (lib_id "power:+24V") (at 50.8 45.72 0) (unit 1)
     (in_bom yes) (on_board yes) (fields_autoplaced)
-    (property "Reference" "#PWR046" (id 0) (at 50.8 49.53 0)
+    (property "Reference" "#PWR021" (id 0) (at 50.8 49.53 0)
       (effects (font (size 1.27 1.27)) hide)
     )
@@
   (symbol (lib_id "Device:D_Zener") (at 68.58 49.53 270) (unit 1)
     (in_bom yes) (on_board yes) (fields_autoplaced)
-    (property "Reference" "D4" (id 0) (at 71.12 48.2599 90)
+    (property "Reference" "D5" (id 0) (at 71.12 48.2599 90)
       (effects (font (size 1.27 1.27)) (justify left))
     )
@@
   (symbol (lib_id "Device:LED") (at 83.82 53.34 90) (unit 1)
     (in_bom yes) (on_board yes) (fields_autoplaced)
-    (property "Reference" "D6" (id 0) (at 87.63 53.6574 90)
+    (property "Reference" "D7" (id 0) (at 87.63 53.6574 90)
       (effects (font (size 1.27 1.27)) (justify right))
     )
@@
   (symbol (lib_id "Device:R") (at 83.82 60.96 180) (unit 1)
     (in_bom yes) (on_board yes)
-    (property "Reference" "R21" (id 0) (at 86.36 60.96 90))
+    (property "Reference" "R5" (id 0) (at 86.36 60.96 90))
     (property "Value" "470R" (id 1) (at 88.9 60.96 90))
     (property "Footprint" "Resistor_SMD:R_0603_1608Metric_Pad0.98x0.95mm_HandSolder" (id 2) (at 85.598 60.96 90)
@@
   (symbol (lib_id "power:GND") (at 83.82 64.77 0) (unit 1)
     (in_bom yes) (on_board yes) (fields_autoplaced)
-    (property "Reference" "#PWR048" (id 0) (at 83.82 71.12 0)
+    (property "Reference" "#PWR023" (id 0) (at 83.82 71.12 0)
       (effects (font (size 1.27 1.27)) hide)
     )
