File: Standardized Subsheets/microcontroller.kicad_sch (KiCad schematic)
At the start: 57 parts, among them J3 Conn_01x02, J4 Conn_01x02, J5 SWD, SW1 SW_SPDT, U2 STM32F105RCTx, U3 SN65HVD230, U4 SN65HVD230, Y1 16MHz

Commit message: updated microcontroller
Parts:
- D2: footprint Global Libraries:SOT95P280X100-6N -> SOT95P280X100-6N
Changed lines of the file:
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@@
       (effects (font (size 1.27 1.27)) (justify right))
     )
-    (property "Footprint" "Global Libraries:SOT95P280X100-6N" (id 2) (at 119.38 115.57 0)
+    (property "Footprint" "SOT95P280X100-6N" (id 2) (at 119.38 115.57 0)
       (effects (font (size 1.27 1.27)) (justify left) hide)
     )
