File: Standardized Subsheets/SEPIC_CAD.kicad_sch (KiCad schematic)
At the start: 25 parts, among them IC1 LM5155DSSR, Q1 CSD18537NQ5A

Commit message: Error Occured
Parts:
- IC1: footprint SON50P200X300X80-13N-D -> Global Libraries:SON50P200X300X80-13N-D
- Q1: footprint CSD19531Q5AT -> Global Libraries:CSD19531Q5AT
Changed lines of the file:
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@@
     (property "Reference" "IC1" (id 0) (at 105.41 63.5 0))
     (property "Value" "LM5155DSSR" (id 1) (at 105.41 66.04 0))
-    (property "Footprint" "SON50P200X300X80-13N-D" (id 2) (at 128.27 77.47 0)
+    (property "Footprint" "Global Libraries:SON50P200X300X80-13N-D" (id 2) (at 128.27 77.47 0)
       (effects (font (size 1.27 1.27)) (justify left) hide)
     )
@@
       (effects (font (size 1.27 1.27)) (justify left))
     )
-    (property "Footprint" "CSD19531Q5AT" (id 2) (at 168.91 76.2 0)
+    (property "Footprint" "Global Libraries:CSD19531Q5AT" (id 2) (at 168.91 76.2 0)
       (effects (font (size 1.27 1.27)) (justify left) hide)
     )
@@
     )
     (path "/3be2f64a-643b-4527-aaf5-307341a81097"
-      (reference "IC1") (unit 1) (value "LM5155DSSR") (footprint "SON50P200X300X80-13N-D")
+      (reference "IC1") (unit 1) (value "LM5155DSSR") (footprint "Global Libraries:SON50P200X300X80-13N-D")
     )
     (path "/465cb822-cddf-441d-8f53-8ae0b192b81a"
@@
     )
     (path "/b6e6a3f1-e3fb-4eaa-bf70-4dd3052bf5ca"
-      (reference "Q1") (unit 1) (value "CSD18537NQ5A") (footprint "CSD19531Q5AT")
+      (reference "Q1") (unit 1) (value "CSD18537NQ5A") (footprint "Global Libraries:CSD19531Q5AT")
     )
     (path "/0bb5cd34-d493-45c4-917f-8c4bd795b455"

Commit message: Lib updates
Parts:
- IC1: footprint Global Libraries:SON50P200X300X80-13N-D -> SON50P200X300X80-13N-D
- Q1: footprint Global Libraries:CSD19531Q5AT -> CSD19531Q5AT
Changed lines of the file:
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@@
     (property "Reference" "IC1" (id 0) (at 105.41 63.5 0))
     (property "Value" "LM5155DSSR" (id 1) (at 105.41 66.04 0))
-    (property "Footprint" "Global Libraries:SON50P200X300X80-13N-D" (id 2) (at 128.27 77.47 0)
+    (property "Footprint" "SON50P200X300X80-13N-D" (id 2) (at 128.27 77.47 0)
       (effects (font (size 1.27 1.27)) (justify left) hide)
     )
@@
       (effects (font (size 1.27 1.27)) (justify left))
     )
-    (property "Footprint" "Global Libraries:CSD19531Q5AT" (id 2) (at 168.91 76.2 0)
+    (property "Footprint" "CSD19531Q5AT" (id 2) (at 168.91 76.2 0)
       (effects (font (size 1.27 1.27)) (justify left) hide)
     )
@@
     )
     (path "/3be2f64a-643b-4527-aaf5-307341a81097"
-      (reference "IC1") (unit 1) (value "LM5155DSSR") (footprint "Global Libraries:SON50P200X300X80-13N-D")
+      (reference "IC1") (unit 1) (value "LM5155DSSR") (footprint "SON50P200X300X80-13N-D")
     )
     (path "/465cb822-cddf-441d-8f53-8ae0b192b81a"
@@
     )
     (path "/b6e6a3f1-e3fb-4eaa-bf70-4dd3052bf5ca"
-      (reference "Q1") (unit 1) (value "CSD18537NQ5A") (footprint "Global Libraries:CSD19531Q5AT")
+      (reference "Q1") (unit 1) (value "CSD18537NQ5A") (footprint "CSD19531Q5AT")
     )
     (path "/0bb5cd34-d493-45c4-917f-8c4bd795b455"
